Commit message: update z-axis of the golf_vehicle

File: golf_vehicle_description/urdf/vehicle.xacro (robot description, xacro)
@@ -10,5 +10,5 @@
     <visual>
       <!--<origin xyz="${vehicle_info['/**']['ros__parameters']['wheel_base']/2.0} 0 0" rpy="${pi/2.0} 0 ${pi/2.0}"/>-->
-      <origin xyz="1.3772 0 -0.3935" rpy="${pi/2.0} 0 -${pi/2.0}"/>
+      <origin xyz="1.3772 0 -0.1" rpy="${pi/2.0} 0 -${pi/2.0}"/>
       <geometry>
         <mesh filename="package://golf_vehicle_description/mesh/golf.fbx" scale="0.01 0.01 0.01"/>

Commit message: Update golf_vehicle_description/urdf/vehicle.xacro
Co-authored-by: Ismet Atabay <56237550+ismetatabay@users.noreply.github.com>

File: golf_vehicle_description/urdf/vehicle.xacro (robot description, xacro)
@@ -10,5 +10,5 @@
     <visual>
       <!--<origin xyz="${vehicle_info['/**']['ros__parameters']['wheel_base']/2.0} 0 0" rpy="${pi/2.0} 0 ${pi/2.0}"/>-->
-      <origin xyz="1.3772 0 -0.1" rpy="${pi/2.0} 0 -${pi/2.0}"/>
+      <origin xyz="1.3772 0 0" rpy="${pi/2.0} 0 -${pi/2.0}"/>
       <geometry>
         <mesh filename="package://golf_vehicle_description/mesh/golf.fbx" scale="0.01 0.01 0.01"/>

Commit message: Update z-axis of the vehicle

File: golf_vehicle_description/urdf/vehicle.xacro (robot description, xacro)
@@ -10,5 +10,5 @@
     <visual>
       <!--<origin xyz="${vehicle_info['/**']['ros__parameters']['wheel_base']/2.0} 0 0" rpy="${pi/2.0} 0 ${pi/2.0}"/>-->
-      <origin xyz="1.3772 0 0" rpy="${pi/2.0} 0 -${pi/2.0}"/>
+      <origin xyz="1.3772 0 0.31" rpy="${pi/2.0} 0 -${pi/2.0}"/>
       <geometry>
         <mesh filename="package://golf_vehicle_description/mesh/golf.fbx" scale="0.01 0.01 0.01"/>

Commit message: add mirror param yaml

File: golf_vehicle_description/urdf/vehicle.xacro (robot description, xacro)
@@ -10,5 +10,5 @@
     <visual>
       <!--<origin xyz="${vehicle_info['/**']['ros__parameters']['wheel_base']/2.0} 0 0" rpy="${pi/2.0} 0 ${pi/2.0}"/>-->
-      <origin xyz="1.3772 0 0.31" rpy="${pi/2.0} 0 -${pi/2.0}"/>
+      <origin xyz="1.3772 0 0.0" rpy="${pi/2.0} 0 -${pi/2.0}"/>
       <geometry>
         <mesh filename="package://golf_vehicle_description/mesh/golf.fbx" scale="0.01 0.01 0.01"/>

Commit message: feat(golf_vehicle_launch): change vehicle's mesh and xacro file
Signed-off-by: Berkay Karaman <brkay54@gmail.com>

File: golf_vehicle_description/urdf/vehicle.xacro (robot description, xacro)
@@ -1,4 +1,4 @@
 <?xml version="1.0"?>
-<robot xmlns:xacro="http://ros.org/wiki/xacro">
+<robot name="golf" xmlns:xacro="http://ros.org/wiki/xacro">
   <!-- load parameter -->
   <xacro:property
@@ -7,12 +7,12 @@
   />
   <!-- vehicle body -->
-  <link name="base_link">
+<link name="base_link">
     <visual>
-      <!--<origin xyz="${vehicle_info['/**']['ros__parameters']['wheel_base']/2.0} 0 0" rpy="${pi/2.0} 0 ${pi/2.0}"/>-->
-      <origin xyz="1.3772 0 0.0" rpy="${pi/2.0} 0 -${pi/2.0}"/>
+      <!--<origin xyz="${vehicle_info['/**']['ros__parameters']['wheel_base']/2.0} 0 0" rpy="0 0 ${pi/2.0}"/>-->
+      <origin xyz="1.3772 0.0 0.0" rpy="0 0 ${pi/2.0}"/>
       <geometry>
-        <mesh filename="package://golf_vehicle_description/mesh/golf.fbx" scale="0.01 0.01 0.01"/>
+        <mesh filename="package://golf_vehicle_description/mesh/golf.dae" scale="1 1 1"/>
       </geometry>
     </visual>
-  </link>
+</link>
 </robot>
